Commit message: Ny package

File: urdf/robot_control.gazebo.xacro (robot description, xacro)
@@ -116,14 +116,14 @@
         <implicitSpringDamper>true</implicitSpringDamper>
     </gazebo>
-    <gazebo reference="left_weel_joint">
+    <!-- <gazebo reference="left_weel_joint">
         <implicitSpringDamper>true</implicitSpringDamper>
     </gazebo>
     <gazebo reference="right_weel_joint">
         <implicitSpringDamper>true</implicitSpringDamper>
-    </gazebo>
+    </gazebo> -->
     <gazebo>
         <plugin filename="libgazebo_ros2_control.so" name="gazebo_ros2_control">
             <robot_sim_type>gazebo_ros2_control/GazeboSystem</robot_sim_type>
-            <parameters>$(find ELE306Prosjekt)/config/controller_config.yaml</parameters>
+            <parameters>$(find robotikk_prosjekt)/config/controller_config.yaml</parameters>
         </plugin>
     </gazebo>
@@ -134,6 +134,6 @@
         <joint name="arm_base_joint">
             <command_interface name="position">
-                <param name="min">-${pi/2}</param>
-                <param name="max">${pi/2}</param>
+                <param name="min">-${pi}</param>
+                <param name="max">${pi}</param>
             </command_interface>
             <state_interface name="position"/>
@@ -159,5 +159,5 @@
             <state_interface name="effort"/>
         </joint>
-        <joint name="wrist_joint">
+        <joint name="wrist_joint_joint">
             <command_interface name="position">
                 <param name="min">-${pi/2}</param>
@@ -170,6 +170,6 @@
         <joint name="gripper_joint">
             <command_interface name="position">
-                <param name="min">-${pi/2}</param>
-                <param name="max">${pi/2}</param>
+                <param name="min">-${pi}</param>
+                <param name="max">${pi}</param>
             </command_interface>
             <state_interface name="position"/>

File: urdf/robot_description.urdf.xacro (robot description, xacro)
@@ -1,6 +1,6 @@
 <?xml version="1.0" ?>
-<robot name="ELE306ProsjektBåt" xmlns:xacro="http://ros.org/wiki/xacro">
-    <xacro:include filename="$(find ELE306Prosjekt)/urdf/common_macros.xacro" />
-    <xacro:include filename="$(find ELE306Prosjekt)/urdf/robot_control.gazebo.xacro" />
+<robot name="robotikk_prosjekt" xmlns:xacro="http://ros.org/wiki/xacro">
+    <xacro:include filename="$(find robotikk_prosjekt)/urdf/common_macros.xacro" />
+    <xacro:include filename="$(find robotikk_prosjekt)/urdf/robot_control.gazebo.xacro" />
     <!-- CTRL + SHIFT + 7 to comment/uncomment marked code! -->
         <!-- <gazebo>
@@ -23,14 +23,14 @@
             <origin xyz="0 0 0" rpy="0 0 0"/>
             <geometry>
-                <mesh filename="$(find ELE306Prosjekt)/meshes/BoatVisualMesh.stl" scale="0.001 0.001 0.001"/>
-            </geometry>
-        </visual>
-        <collision>
-            <origin xyz="0 0 0" rpy="0 0 0"/>
-            <geometry>
-                <mesh filename="$(find ELE306Prosjekt)/meshes/BoatColitionMesh.stl" scale="0.001 0.001 0.001"/>
-            </geometry>
-        </collision>
-        <xacro:inertial_box length="1.0" width="0.400" height="0.300" density="${density_pla}">
+                <mesh filename="$(find robotikk_prosjekt)/meshes/BoatVisualMesh.stl" scale="0.001 0.001 0.001"/>
+            </geometry>
+        </visual>
+        <collision>
+            <origin xyz="0 0 0" rpy="0 0 0"/>
+            <geometry>
+                <mesh filename="$(find robotikk_prosjekt)/meshes/BoatColitionMesh.stl" scale="0.001 0.001 0.001"/>
+            </geometry>
+        </collision>
+        <xacro:inertial_box length="1.0" width="0.400" height="0.300" density="${density_pla*10}">
             <origin xyz="0 0 0" rpy="0 0 0"/>
         </xacro:inertial_box>
@@ -50,5 +50,5 @@
             <origin xyz="0 0 0" rpy="0 0 0"/>
             <geometry>
-                <mesh filename="$(find ELE306Prosjekt)/meshes/BaseJoint.stl" scale="0.001 0.001 0.001"/>
+                <mesh filename="$(find robotikk_prosjekt)/meshes/BaseJoint.stl" scale="0.001 0.001 0.001"/>
             </geometry>
         </visual>
@@ -71,5 +71,5 @@
         <axis xyz="0 0 1" rpy="0 0 0"/>
         <limit effort="1000" velocity="1000"/>
-        <dynamics damping="0.7" friction="100.0"/>
+        <dynamics damping="0.7" friction="1.0"/>
     </joint>
     <link name="left_wheel_link">
@@ -77,11 +77,11 @@
             <origin xyz="0 0 0" rpy="0 0 0"/>
             <geometry>
-                <cylinder length="0.1" radius="${0.2/2}" />
-            </geometry>
-        </visual>
-        <collision>
-            <origin xyz="0 0 0" rpy="0 0 0"/>
-            <geometry>
-                <cylinder length="0.1" radius="${0.2/2}" />
+                <cylinder length="0.1" radius="${0.201/2}" />
+            </geometry>
+        </visual>
+        <collision>
+            <origin xyz="0 0 0" rpy="0 0 0"/>
+            <geometry>
+                <cylinder length="0.1" radius="${0.201/2}" />
             </geometry>
         </collision>
@@ -93,10 +93,10 @@
     <!-- ==================================== -->
     <joint type="continuous" name="right_wheel_joint">
-        <origin xyz="0 -${0.2 + 0.1 / 2} 0.25" rpy="${pi/2} 0 0"/>
+        <origin xyz="0 -${0.2 + 0.1 / 2} 0.25" rpy="-${pi/2} 0 0"/>
         <child link="right_wheel_link"/>
         <parent link="mobile_boat_link"/>
         <axis xyz="0 0 1" rpy="0 0 0"/>
         <limit effort="1000" velocity="1000"/>
-        <dynamics damping="0.7" friction="100.0"/>
+        <dynamics damping="0.7" friction="1.0"/>
     </joint>
     <link name="right_wheel_link">
@@ -104,11 +104,11 @@
             <origin xyz="0 0 0" rpy="0 0 0"/>
             <geometry>
-                <cylinder length="0.1" radius="${0.2/2}" />
-            </geometry>
-        </visual>
-        <collision>
-            <origin xyz="0 0 0" rpy="0 0 0"/>
-            <geometry>
-                <cylinder length="0.1" radius="${0.2/2}" />
+                <cylinder length="0.1" radius="${0.205/2}" />
+            </geometry>
+        </visual>
+        <collision>
+            <origin xyz="0 0 0" rpy="0 0 0"/>
+            <geometry>
+                <cylinder length="0.1" radius="${0.205/2}" />
             </geometry>
         </collision>
@@ -131,5 +131,5 @@
             <origin xyz="0 0 0" rpy="0 0 0"/>
             <geometry>
-                <mesh filename="$(find ELE306Prosjekt)/meshes/Arm1.stl" scale="0.001 0.001 0.001"/>
+                <mesh filename="$(find robotikk_prosjekt)/meshes/Arm1.stl" scale="0.001 0.001 0.001"/>
             </geometry>
         </visual>
@@ -158,5 +158,5 @@
             <origin xyz="0 0 0" rpy="0 0 0"/>
             <geometry>
-                <mesh filename="$(find ELE306Prosjekt)/meshes/Arm2.stl" scale="0.001 0.001 0.001"/>
+                <mesh filename="$(find robotikk_prosjekt)/meshes/Arm2.stl" scale="0.001 0.001 0.001"/>
             </geometry>
         </visual>
@@ -185,5 +185,5 @@
             <origin xyz="0 0 0" rpy="0 0 0"/>
             <geometry>
-                <mesh filename="$(find ELE306Prosjekt)/meshes/WristJoint.stl" scale="0.001 0.001 0.001"/>
+                <mesh filename="$(find robotikk_prosjekt)/meshes/WristJoint.stl" scale="0.001 0.001 0.001"/>
             </geometry>
         </visual>
@@ -212,5 +212,5 @@
             <origin xyz="0 0 0" rpy="0 0 0"/>
             <geometry>
-                <mesh filename="$(find ELE306Prosjekt)/meshes/Gripper.stl" scale="0.001 0.001 0.001"/>
+                <mesh filename="$(find robotikk_prosjekt)/meshes/Gripper.stl" scale="0.001 0.001 0.001"/>
             </geometry>
         </visual>
